File: PmodICSIF.kicad_pcb (KiCad board)
At the start: 2 copper layers, 28 parts, among them IC1 SN74LV1T125DBVR, IC2 SN74LV1T125DBVR, IC3 SN74LV1T125DBVR, IC4 SN74LV1T125DBVR, IC5 MC7805CDTRKG, IC6 SN74LV1T125DBVR, IC7 SN74LV1T125DBVR, J1 Conn_02x06_Top_Bottom, J2 Conn_01x02, J3 Conn_01x03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

Commit message: drawed
Parts:
- C1, C2, C4, C5, C6, C7: moved to B.Cu
- J1: footprint Connectors_Samtec:SDL-112-X-XX_2x06 -> kicad-pmod:pmod_pin_array_6x2
- moved J2 114.8 mm to (119.0, 71.2), turned to 270 degrees
- moved C3 100.2 mm to (120.8, 81.5), turned to 180 degrees
- moved IC5 86.1 mm to (120.3, 91.8), turned to 270 degrees
- moved C6 68.6 mm to (88.2, 97.9), turned to 0 degrees
- moved IC6 68.4 mm to (87.0, 97.2), turned to 180 degrees
- moved C7 67.5 mm to (88.1, 85.6), turned to 0 degrees
- moved IC7 65.2 mm to (87.0, 84.6), turned to 180 degrees
- moved R3 56.6 mm to (93.5, 97.2), turned to 180 degrees
- moved R4 52.5 mm to (93.6, 84.6), turned to 180 degrees
- moved C1 51.9 mm to (85.8, 90.8), turned to 180 degrees
- moved IC1 51.8 mm to (87.0, 91.6)
- moved IC3 50.2 mm to (94.3, 93.5)
- moved C4 49.5 mm to (93.1, 93.5), turned to 180 degrees
- moved C2 49.3 mm to (86.2, 78.0), turned to 180 degrees
- moved R5 49.3 mm to (100.2, 92.5)
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Connections:
- C1 pad 2: GNDD -> GND
- C2 pad 2: GNDD -> GND
- C3 pad 2: GNDA -> GND
- C4 pad 2: GNDA -> GND
- C5 pad 2: GNDA -> GND
- C6 pad 2: GNDD -> GND
- C7 pad 2: GNDD -> GND
- D3 pad 2: GNDA -> GND
- D4 pad 2: GNDA -> GND
- IC1 pad 3: GNDD -> GND
- IC2 pad 3: GNDD -> GND
- IC3 pad 3: GNDA -> GND
- IC4 pad 3: GNDA -> GND
- IC5 pad 2: GNDA -> GND
- IC5 pad 4: GNDA -> GND
- IC6 pad 3: GNDD -> GND
- IC7 pad 3: GNDD -> GND
- J2 pad 2: GNDA -> GND
- J3 pad 3: GNDA -> GND
- J4 pad 3: GNDA -> GND
Other:
- net class Bold added: clearance 0.4, trace_width 0.5, via_dia 0.8, via_drill 0.4
- rule trace_min: 0.2 -> 0.1524
- rule via_min_drill: 0.3 -> 0.2
- rule via_min_size: 0.4 -> 0.5
